Commit message: Updated code for grasp planning

File: franka_description/end_effectors/common/franka_hand.xacro (robot description, xacro)
@@ -126,5 +126,4 @@
       <axis xyz="0 1 0" />
       <limit effort="100" lower="0.0" upper="0.04" velocity="0.2" />
-      <mimic joint="${ee_prefix}finger_joint1" />
       <dynamics damping="0.3" />
     </joint>

File: franka_description/robots/common/franka_arm.ros2_control.xacro (robot description, xacro)
@@ -60,4 +60,5 @@
       <xacro:if value="${gazebo and hand}">
         <xacro:configure_joint joint_name="${arm_prefix}${arm_id}_finger_joint1" initial_position="0.0" />
+        <xacro:configure_joint joint_name="${arm_prefix}${arm_id}_finger_joint2" initial_position="0.0" />
       </xacro:if>
       <xacro:macro name="general_purpose_io" params="prefix command_interface index">
